File: daisy_01/daisy_01.kicad_pcb (KiCad board)
At the start: 2 copper layers, 106.7 x 30.5 mm, 17 parts, among them J1 AudioInput, J2 AudioOutput1, J3 AudioOutput2, Q1 PN2222A, SW1 SW_SPST, SW2 RotaryEncoder_Switch

Commit message: update
Routing:
- net GND: track 180.3 -> 236.4 mm
Changed lines of the file:
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@@
   (segment (start 173.99 106.68) (end 176.49 109.18) (width 0.25) (layer "F.Cu") (net 3))
   (segment (start 111.76 104.14) (end 104.14 111.76) (width 0.25) (layer "F.Cu") (net 3))
+  (segment (start 149.86 127) (end 114.3 127) (width 0.25) (layer "B.Cu") (net 3))
+  (segment (start 152.4 129.54) (end 149.86 127) (width 0.25) (layer "B.Cu") (net 3))
+  (segment (start 114.3 127) (end 104.14 116.84) (width 0.25) (layer "B.Cu") (net 3))
+  (segment (start 104.14 116.84) (end 104.14 114.3) (width 0.25) (layer "B.Cu") (net 3))
   (segment (start 203.2 121.92) (end 200.66 121.92) (width 0.25) (layer "F.Cu") (net 4))
   (segment (start 205.74 124.46) (end 203.2 121.92) (width 0.25) (layer "F.Cu") (net 4))
