File: daisy_01/daisy_01.kicad_pcb (KiCad board)
At the start: 2 copper layers, 165.1 x 99.1 mm, 16 parts, among them J1 AudioInput, J2 AudioOutput1, J3 AudioOutput2, Q1 PN2222A, SW1 SW_SPST

Commit message: update
Parts:
- moved RV4 129.1 mm to (116.8, 106.7), turned to -90 degrees
- moved RV3 116.0 mm to (134.6, 106.7), turned to -90 degrees
- moved RV2 105.7 mm to (152.4, 106.7), turned to -90 degrees
- moved RV1 98.8 mm to (170.1, 106.7), turned to -90 degrees
- moved A1 87.2 mm to (104.1, 129.5), turned to 90 degrees
- moved C1 78.9 mm to (170.2, 116.8)
- moved J1 76.2 mm to (185.4, 119.4)
- moved R1 72.7 mm to (196.8, 124.5)
- moved J2 66.1 mm to (185.4, 124.5)
- moved SW1 64.1 mm to (198.1, 129.5)
- moved BT1 61.1 mm to (198.1, 119.4)
- moved J3 61.0 mm to (185.4, 129.5)
- moved C2 58.5 mm to (162.6, 114.3)
- moved D1 50.7 mm to (203.2, 106.7)
- moved R2 46.6 mm to (161.3, 129.5)
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- renumbered R3 to R2
Other:
- board size 165.1 x 99.1 mm -> 109.2 x 30.5 mm

Commit message: update
Parts:
- removed A1: Device_Audio_Electrosmith_Daisy_Seed_Rev4, Daisy_Electrosmith:Device_Audio_Electrosmith_Daisy_Seed
- added SW2: RotaryEncoder_Switch, Rotary_Encoder:RotaryEncoder_Alps_EC11E-Switch_Vertical_H20mm, F.Cu at (180.7, 104.2)
- added U1: ~, Library_electrosmith:Device_Audio_Electrosmith_Daisy_Seed, F.Cu at (104.1, 129.5)
- moved C1 26.1 mm to (193.0, 129.5), turned to 90 degrees
- moved C2 25.9 mm to (188.0, 119.4)
- moved R2 25.5 mm to (186.7, 127.0), turned to 180 degrees
- moved J1 20.5 mm to (165.1, 116.8), turned to 180 degrees
- moved J2 20.5 mm to (165.1, 121.9), turned to 180 degrees
- moved J3 20.5 mm to (165.1, 127.0), turned to 180 degrees
- moved Q1 18.0 mm to (180.3, 119.4), turned to 180 degrees
- moved BT1 12.7 mm to (205.7, 129.5), turned to 90 degrees
- moved R1 11.7 mm to (205.7, 116.8), turned to 180 degrees
- moved SW1 8.03 mm to (200.7, 121.9), turned to 180 degrees
Routing:
- net GND: track 0.00 -> 137.0 mm
- net +9V: track 0.00 -> 109.1 mm
- net /A_PWR3.3: track 0.00 -> 82.8 mm
- net Net-(U1-A3/D18): track 0.00 -> 28.6 mm
- net Net-(J1-PadT): track 0.00 -> 25.6 mm
- net Net-(U1-A5/D21): track 0.00 -> 23.5 mm
- net Net-(Q1-B): track 0.00 -> 19.9 mm
- net Net-(Q1-E): track 0.00 -> 18.8 mm
- net Net-(U1-Audio_Out_1): track 0.00 -> 18.4 mm
- net Net-(U1-Audio_Out_2): track 0.00 -> 13.8 mm
- net Net-(U1-A4/D19): track 0.00 -> 13.3 mm
- net Net-(D1-A): track 0.00 -> 10.2 mm
- net Net-(U1-A5/D20): track 0.00 -> 9.71 mm
- net Net-(BT1--): track 0.00 -> 6.13 mm

Commit message: update
Routing:
- net GND: track 137.0 -> 191.5 mm
Changed lines of the file:
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@@
   (segment (start 152.36 106.64) (end 152.36 106.68) (width 0.25) (layer "B.Cu") (net 1))
   (segment (start 134.62 106.68) (end 137.16 104.14) (width 0.25) (layer "B.Cu") (net 1))
-  (segment (start 111.76 119.38) (end 106.68 114.3) (width 0.25) (layer "F.Cu") (net 2))
   (segment (start 177.8 125.73) (end 179.07 127) (width 0.25) (layer "F.Cu") (net 2))
   (segment (start 180.34 127) (end 179.07 127) (width 0.25) (layer "F.Cu") (net 2))
   (segment (start 182.92 129.5) (end 182.88 129.54) (width 0.25) (layer "F.Cu") (net 2))
+  (segment (start 193.04 129.5) (end 182.92 129.5) (width 0.25) (layer "F.Cu") (net 2))
+  (segment (start 111.76 119.38) (end 106.68 114.3) (width 0.25) (layer "F.Cu") (net 2))
   (segment (start 177.8 119.38) (end 111.76 119.38) (width 0.25) (layer "F.Cu") (net 2))
-  (segment (start 193.04 129.5) (end 182.92 129.5) (width 0.25) (layer "F.Cu") (net 2))
   (segment (start 205.74 129.54) (end 193.08 129.54) (width 0.25) (layer "F.Cu") (net 2))
   (segment (start 193.08 129.54) (end 193.04 129.5) (width 0.25) (layer "F.Cu") (net 2))
@@
   (segment (start 193.04 119.38) (end 190.5 119.38) (width 0.25) (layer "F.Cu") (net 3))
   (segment (start 195.58 121.92) (end 193.04 124.46) (width 0.25) (layer "F.Cu") (net 3))
+  (segment (start 111.76 121.92) (end 104.14 114.3) (width 0.25) (layer "F.Cu") (net 3))
   (segment (start 127.08 109.22) (end 129.62 106.68) (width 0.25) (layer "F.Cu") (net 3))
   (segment (start 144.82 104.14) (end 147.36 106.68) (width 0.25) (layer "F.Cu") (net 3))
@@
   (segment (start 106.68 106.68) (end 111.8 106.68) (width 0.25) (layer "F.Cu") (net 3))
   (segment (start 104.18 114.3) (end 104.14 114.3) (width 0.25) (layer "F.Cu") (net 3))
+  (segment (start 144.78 121.92) (end 111.76 121.92) (width 0.25) (layer "F.Cu") (net 3))
+  (segment (start 152.4 129.54) (end 144.78 121.92) (width 0.25) (layer "F.Cu") (net 3))
   (segment (start 132.08 104.14) (end 144.82 104.14) (width 0.25) (layer "F.Cu") (net 3))
   (segment (start 132.08 109.14) (end 132.08 109.22) (width 0.25) (layer "F.Cu") (net 3))

Commit message: update
Parts:
- moved C2 3.59 mm to (185.5, 121.9)
- moved Q1 3.59 mm to (177.8, 121.9)
- moved R2 3.59 mm to (184.2, 129.5)
- moved SW2 3.31 mm to (178.5, 106.7)
- moved D1 2.54 mm to (200.7, 106.7)
- moved J1 2.54 mm to (165.1, 119.4)
- moved J2 2.54 mm to (165.1, 124.5)
- moved J3 2.54 mm to (165.1, 129.5)
Connections:
- RV1 pad 1: /A_PWR3.3 -> GND
- RV1 pad 3: GND -> /A_PWR3.3
- RV2 pad 1: /A_PWR3.3 -> GND
- RV2 pad 3: GND -> /A_PWR3.3
- RV3 pad 1: /A_PWR3.3 -> GND
- RV3 pad 3: GND -> /A_PWR3.3
- RV4 pad 1: /A_PWR3.3 -> GND
- RV4 pad 3: GND -> /A_PWR3.3
Routing:
- net Net-(U1-A2/D17): track 0.00 -> 53.5 mm
- net Net-(U1-A1/D16): track 0.00 -> 33.4 mm
- net Net-(U1-A0/D15): track 0.00 -> 31.8 mm
- net /A_PWR3.3: track 82.8 -> 64.4 mm
- net GND: track 191.5 -> 180.3 mm
- net +9V: track 109.1 -> 114.6 mm
- net Net-(Q1-E): track 18.8 -> 22.4 mm
- net Net-(Q1-B): track 19.9 -> 18.5 mm
- net Net-(D1-A): track 10.2 -> 11.2 mm
- net Net-(J1-PadT): track 25.6 -> 24.5 mm
- net Net-(U1-Audio_Out_2): track 13.8 -> 14.8 mm
- net Net-(U1-Audio_Out_1): track 18.4 -> 17.3 mm
Other:
- board size 109.2 x 30.5 mm -> 106.7 x 30.5 mm

Commit message: update
Parts:
- moved J3 39.5 mm to (204.5, 127.0), turned to -90 degrees
- moved SW1 38.2 mm to (162.6, 124.5)
- moved BT1 38.1 mm to (167.6, 129.5)
- moved J1 31.4 mm to (195.6, 127.0), turned to -90 degrees
- moved J2 21.7 mm to (186.7, 127.0), turned to -90 degrees
- moved C1 17.7 mm to (176.5, 123.2)
- moved C2 17.3 mm to (168.9, 116.8)
- moved Q1 16.1 mm to (162.6, 116.8)
- moved R2 2.54 mm to (181.6, 129.5)
Routing:
- net Net-(U1-Audio_Out_2): track 14.8 -> 56.0 mm
- net +9V: track 114.6 -> 84.0 mm
- net Net-(J1-PadT): track 24.5 -> 54.7 mm
- net Net-(U1-Audio_Out_1): track 17.3 -> 40.7 mm
- net Net-(Q1-E): track 22.4 -> 36.5 mm
- net Net-(Q1-B): track 18.5 -> 30.4 mm
- net GND: track 180.3 -> 176.6 mm
- net Net-(U1-A3/D18): track 28.6 -> 30.4 mm
- net Net-(BT1--): track 6.13 -> 5.08 mm
- net Net-(U1-A2/D17): track 53.5 -> 52.5 mm
- net /A_PWR3.3: track 64.4 -> 65.1 mm
