File: daisy_01/daisy_01.kicad_pcb (KiCad board)
At the start: 2 copper layers, 106.7 x 30.5 mm, 17 parts, among them J1 AudioInput, J2 AudioOutput1, J3 AudioOutput2, Q1 PN2222A, SW1 SW_SPST, SW2 RotaryEncoder_Switch

Commit message: update
Routing:
- net GND: track 180.3 -> 0.00 mm
- net +9V: track 114.6 -> 0.00 mm
- net /A_PWR3.3: track 64.4 -> 0.00 mm
- net Net-(U1-A2/D17): track 53.5 -> 0.00 mm
- net Net-(U1-A1/D16): track 33.4 -> 0.00 mm
- net Net-(U1-A0/D15): track 31.8 -> 0.00 mm
- net Net-(U1-A3/D18): track 28.6 -> 0.00 mm
- net Net-(J1-PadT): track 24.5 -> 0.00 mm
- net Net-(U1-A5/D21): track 23.5 -> 0.00 mm
- net Net-(Q1-E): track 22.4 -> 0.00 mm
- net Net-(Q1-B): track 18.5 -> 0.00 mm
- net Net-(U1-Audio_Out_1): track 17.3 -> 0.00 mm
- net Net-(U1-Audio_Out_2): track 14.8 -> 0.00 mm
- net Net-(U1-A4/D19): track 13.3 -> 0.00 mm
- net Net-(D1-A): track 11.2 -> 0.00 mm
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Changed lines of the file:
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@@
   (gr_rect (start 101.6 101.6) (end 208.28 132.08)
     (stroke (width 0.1) (type default)) (fill none) (layer "Edge.Cuts"))
-  (segment (start 152.4 114.3) (end 152.4 111.72) (width 0.25) (layer "F.Cu") (net 1))
-  (segment (start 152.4 111.72) (end 147.36 106.68) (width 0.25) (layer "F.Cu") (net 1))
-  (segment (start 165.14 106.68) (end 157.52 114.3) (width 0.25) (layer "F.Cu") (net 1))
-  (segment (start 157.52 114.3) (end 152.4 114.3) (width 0.25) (layer "F.Cu") (net 1))
-  (segment (start 114.3 109.22) (end 127.08 109.22) (width 0.25) (layer "B.Cu") (net 1))
-  (segment (start 130.81 105.49) (end 129.62 106.68) (width 0.25) (layer "B.Cu") (net 1))
-  (segment (start 146.09 105.41) (end 130.81 105.41) (width 0.25) (layer "B.Cu") (net 1))
-  (segment (start 114.3 109.18) (end 114.3 109.22) (width 0.25) (layer "B.Cu") (net 1))
-  (segment (start 127.08 109.22) (end 129.62 106.68) (width 0.25) (layer "B.Cu") (net 1))
-  (segment (start 130.81 105.41) (end 130.81 105.49) (width 0.25) (layer "B.Cu") (net 1))
-  (segment (start 111.8 106.68) (end 114.3 109.18) (width 0.25) (layer "B.Cu") (net 1))
-  (segment (start 147.36 106.68) (end 146.09 105.41) (width 0.25) (layer "B.Cu") (net 1))
-  (segment (start 176.53 129.54) (end 175.26 128.27) (width 0.25) (layer "F.Cu") (net 2))
-  (segment (start 193.08 129.54) (end 193.04 129.5) (width 0.25) (layer "F.Cu") (net 2))
-  (segment (start 177.8 130.81) (end 176.53 129.54) (width 0.25) (layer "F.Cu") (net 2))
-  (segment (start 193.04 129.5) (end 191.73 130.81) (width 0.25) (layer "F.Cu") (net 2))
-  (segment (start 205.74 129.54) (end 193.08 129.54) (width 0.25) (layer "F.Cu") (net 2))
-  (segment (start 175.26 128.27) (end 175.26 121.92) (width 0.25) (layer "F.Cu") (net 2))
-  (segment (start 191.73 130.81) (end 177.8 130.81) (width 0.25) (layer "F.Cu") (net 2))
-  (segment (start 151.13 123.19) (end 115.57 123.19) (width 0.25) (layer "B.Cu") (net 2))
-  (segment (start 115.57 123.19) (end 106.68 114.3) (width 0.25) (layer "B.Cu") (net 2))
-  (segment (start 173.99 127) (end 154.94 127) (width 0.25) (layer "B.Cu") (net 2))
-  (segment (start 176.53 129.54) (end 173.99 127) (width 0.25) (layer "B.Cu") (net 2))
-  (segment (start 154.94 127) (end 151.13 123.19) (width 0.25) (layer "B.Cu") (net 2))
-  (segment (start 198.04 106.68) (end 200.66 106.68) (width 0.25) (layer "F.Cu") (net 3))
-  (segment (start 181.04 111.68) (end 193.04 111.68) (width 0.25) (layer "F.Cu") (net 3))
-  (segment (start 166.172 131.008) (end 153.868 131.008) (width 0.25) (layer "F.Cu") (net 3))
-  (segment (start 167.64 124.46) (end 167.64 129.54) (width 0.25) (layer "F.Cu") (net 3))
-  (segment (start 132.08 109.22) (end 119.38 109.22) (width 0.25) (layer "F.Cu") (net 3))
-  (segment (start 195.58 121.92) (end 193.04 119.38) (width 0.25) (layer "F.Cu") (net 3))
-  (segment (start 152.36 106.68) (end 152.36 105.37) (width 0.25) (layer "F.Cu") (net 3))
-  (segment (start 170.14 106.68) (end 173.99 106.68) (width 0.25) (layer "F.Cu") (net 3))
-  (segment (start 153.868 131.008) (end 152.4 129.54) (width 0.25) (layer "F.Cu") (net 3))
-  (segment (start 137.16 104.14) (end 134.62 106.68) (width 0.25) (layer "F.Cu") (net 3))
-  (segment (start 116.8 106.68) (end 116.8 106.72) (width 0.25) (layer "F.Cu") (net 3))
-  (segment (start 167.64 129.54) (end 166.172 131.008) (width 0.25) (layer "F.Cu") (net 3))
-  (segment (start 167.64 119.38) (end 167.64 124.46) (width 0.25) (layer "F.Cu") (net 3))
-  (segment (start 178.54 109.18) (end 181.04 111.68) (width 0.25) (layer "F.Cu") (net 3))
-  (segment (start 116.8 106.68) (end 114.26 104.14) (width 0.25) (layer "F.Cu") (net 3))
-  (segment (start 151.13 104.14) (end 137.16 104.14) (width 0.25) (layer "F.Cu") (net 3))
-  (segment (start 134.62 106.68) (end 132.08 109.22) (width 0.25) (layer "F.Cu") (net 3))
-  (segment (start 195.58 124.46) (end 193.04 127) (width 0.25) (layer "F.Cu") (net 3))
-  (segment (start 104.14 111.76) (end 104.14 114.3) (width 0.25) (layer "F.Cu") (net 3))
-  (segment (start 193.04 119.38) (end 193.04 111.68) (width 0.25) (layer "F.Cu") (net 3))
-  (segment (start 170.14 105.37) (end 170.14 106.68) (width 0.25) (layer "F.Cu") (net 3))
-  (segment (start 119.38 109.22) (end 116.84 106.68) (width 0.25) (layer "F.Cu") (net 3))
-  (segment (start 170.14 106.68) (end 170.14 116.88) (width 0.25) (layer "F.Cu") (net 3))
-  (segment (start 176.49 109.18) (end 178.54 109.18) (width 0.25) (layer "F.Cu") (net 3))
-  (segment (start 114.26 104.14) (end 111.76 104.14) (width 0.25) (layer "F.Cu") (net 3))
-  (segment (start 193.04 111.68) (end 198.04 106.68) (width 0.25) (layer "F.Cu") (net 3))
-  (segment (start 195.58 121.92) (end 195.58 124.46) (width 0.25) (layer "F.Cu") (net 3))
-  (segment (start 187.96 121.92) (end 193.04 127) (width 0.25) (layer "F.Cu") (net 3))
-  (segment (start 152.36 106.68) (end 161.29 106.68) (width 0.25) (layer "F.Cu") (net 3))
-  (segment (start 163.83 104.14) (end 168.91 104.14) (width 0.25) (layer "F.Cu") (net 3))
-  (segment (start 170.14 116.88) (end 167.64 119.38) (width 0.25) (layer "F.Cu") (net 3))
-  (segment (start 116.84 106.68) (end 116.8 106.68) (width 0.25) (layer "F.Cu") (net 3))
-  (segment (start 161.29 106.68) (end 163.83 104.14) (width 0.25) (layer "F.Cu") (net 3))
-  (segment (start 152.36 106.72) (end 152.36 106.68) (width 0.25) (layer "F.Cu") (net 3))
-  (segment (start 152.36 105.37) (end 151.13 104.14) (width 0.25) (layer "F.Cu") (net 3))
-  (segment (start 168.91 104.14) (end 170.14 105.37) (width 0.25) (layer "F.Cu") (net 3))
-  (segment (start 173.99 106.68) (end 176.49 109.18) (width 0.25) (layer "F.Cu") (net 3))
-  (segment (start 111.76 104.14) (end 104.14 111.76) (width 0.25) (layer "F.Cu") (net 3))
-  (segment (start 203.2 121.92) (end 200.66 121.92) (width 0.25) (layer "F.Cu") (net 4))
-  (segment (start 205.74 124.46) (end 203.2 121.92) (width 0.25) (layer "F.Cu") (net 4))
-  (segment (start 177.145 120.65) (end 176.53 121.265) (width 0.25) (layer "F.Cu") (net 5))
-  (segment (start 185.46 128.23) (end 185.46 121.92) (width 0.25) (layer "F.Cu") (net 5))
-  (segment (start 185.46 121.92) (end 185.42 121.92) (width 0.25) (layer "F.Cu") (net 5))
-  (segment (start 176.53 121.265) (end 176.53 121.92) (width 0.25) (layer "F.Cu") (net 5))
-  (segment (start 185.42 121.92) (end 184.15 120.65) (width 0.25) (layer "F.Cu") (net 5))
-  (segment (start 184.15 120.65) (end 177.145 120.65) (width 0.25) (layer "F.Cu") (net 5))
-  (segment (start 184.15 129.54) (end 185.46 128.23) (width 0.25) (layer "F.Cu") (net 5))
-  (segment (start 182.88 116.84) (end 177.8 121.92) (width 0.25) (layer "B.Cu") (net 6))
-  (segment (start 198.12 116.84) (end 182.88 116.84) (width 0.25) (layer "B.Cu") (net 6))
-  (segment (start 205.74 109.22) (end 205.74 116.84) (width 0.25) (layer "F.Cu") (net 7))
-  (segment (start 203.2 106.68) (end 205.74 109.22) (width 0.25) (layer "F.Cu") (net 7))
-  (segment (start 162.56 119.38) (end 152.4 119.38) (width 0.25) (layer "F.Cu") (net 8))
-  (segment (start 152.4 119.38) (end 142.24 129.54) (width 0.25) (layer "F.Cu") (net 8))
-  (segment (start 152.4 124.46) (end 147.32 129.54) (width 0.25) (layer "F.Cu") (net 9))
-  (segment (start 162.56 124.46) (end 152.4 124.46) (width 0.25) (layer "F.Cu") (net 9))
-  (segment (start 162.56 129.54) (end 160.02 127) (width 0.25) (layer "F.Cu") (net 10))
-  (segment (start 152.4 127) (end 149.86 129.54) (width 0.25) (layer "F.Cu") (net 10))
-  (segment (start 160.02 127) (end 152.4 127) (width 0.25) (layer "F.Cu") (net 10))
-  (segment (start 167.64 106.68) (end 165.1 109.22) (width 0.25) (layer "B.Cu") (net 11))
-  (segment (start 165.1 109.22) (end 153.67 109.22) (width 0.25) (layer "B.Cu") (net 11))
-  (segment (start 151.13 111.76) (end 144.78 111.76) (width 0.25) (layer "B.Cu") (net 11))
-  (segment (start 153.67 109.22) (end 151.13 111.76) (width 0.25) (layer "B.Cu") (net 11))
-  (segment (start 144.78 111.76) (end 142.24 114.3) (width 0.25) (layer "B.Cu") (net 11))
-  (segment (start 146.05 110.49) (end 143.51 110.49) (width 0.25) (layer "B.Cu") (net 12))
-  (segment (start 149.86 106.68) (end 146.05 110.49) (width 0.25) (layer "B.Cu") (net 12))
-  (segment (start 143.51 110.49) (end 139.7 114.3) (width 0.25) (layer "B.Cu") (net 12))
-  (segment (start 132.12 109.26) (end 137.16 114.3) (width 0.25) (layer "B.Cu") (net 13))
-  (segment (start 132.12 106.68) (end 132.12 109.26) (width 0.25) (layer "B.Cu") (net 13))
-  (segment (start 114.3 106.68) (end 118.11 110.49) (width 0.25) (layer "F.Cu") (net 14))
-  (segment (start 118.11 110.49) (end 130.81 110.49) (width 0.25) (layer "F.Cu") (net 14))
-  (segment (start 130.81 110.49) (end 134.62 114.3) (width 0.25) (layer "F.Cu") (net 14))
-  (segment (start 174.73 110.49) (end 153.67 110.49) (width 0.25) (layer "B.Cu") (net 31))
-  (segment (start 153.67 110.49) (end 149.86 114.3) (width 0.25) (layer "B.Cu") (net 31))
-  (segment (start 178.54 106.68) (end 174.73 110.49) (width 0.25) (layer "B.Cu") (net 31))
-  (segment (start 148.59 115.57) (end 147.32 114.3) (width 0.25) (layer "B.Cu") (net 32))
-  (segment (start 174.65 115.57) (end 148.59 115.57) (width 0.25) (layer "B.Cu") (net 32))
-  (segment (start 178.54 111.68) (end 174.65 115.57) (width 0.25) (layer "B.Cu") (net 32))
-  (segment (start 175.26 116.84) (end 147.32 116.84) (width 0.25) (layer "B.Cu") (net 33))
-  (segment (start 193.04 106.68) (end 185.42 106.68) (width 0.25) (layer "B.Cu") (net 33))
-  (segment (start 147.32 116.84) (end 144.78 114.3) (width 0.25) (layer "B.Cu") (net 33))
-  (segment (start 185.42 106.68) (end 175.26 116.84) (width 0.25) (layer "B.Cu") (net 33))
 )

Commit message: update
Parts:
- SW2: footprint Rotary_Encoder:RotaryEncoder_Alps_EC11E-Switch_Vertical_H20mm -> personal_footprints:ec11_encoder_mio
- moved R1 25.6 mm to (180.3, 113.6)
- moved D1 19.1 mm to (181.6, 108.0)
- moved J3 19.1 mm to (185.4, 126.3)
- moved J1 15.3 mm to (180.3, 126.3)
- moved R2 14.0 mm to (167.6, 128.8), turned to 0 degrees
- moved SW2 13.3 mm to (177.8, 120.0)
- moved J2 10.9 mm to (185.4, 116.1)
- moved C1 6.38 mm to (170.2, 123.7)
- moved RV4 5.25 mm to (111.7, 108.0)
- moved BT1 5.13 mm to (162.6, 128.8), turned to 180 degrees
- moved C2 4.32 mm to (165.1, 114.9)
- moved RV3 2.88 mm to (132.1, 108.0)
- moved Q1 2.63 mm to (160.0, 116.1)
- moved RV2 1.86 mm to (151.1, 108.0)
- moved RV1 1.36 mm to (170.1, 108.0)
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Routing:
- net GND: track 0.00 -> 152.0 mm
- net +9V: track 0.00 -> 84.3 mm
- net /A_PWR3.3: track 0.00 -> 65.1 mm
- net Net-(U1-Audio_Out_1): track 0.00 -> 45.1 mm
- net Net-(J1-PadT): track 0.00 -> 39.8 mm
- net Net-(U1-Audio_Out_2): track 0.00 -> 38.1 mm
- net Net-(U1-A1/D16): track 0.00 -> 37.6 mm
- net Net-(U1-A0/D15): track 0.00 -> 32.2 mm
- net Net-(U1-A2/D17): track 0.00 -> 32.1 mm
- net Net-(U1-A5/D21): track 0.00 -> 27.7 mm
- net Net-(U1-A3/D18): track 0.00 -> 27.7 mm
- net Net-(Q1-B): track 0.00 -> 23.9 mm
- net Net-(Q1-E): track 0.00 -> 13.8 mm
- net Net-(U1-A4/D19): track 0.00 -> 11.2 mm
- net Net-(U1-A5/D20): track 0.00 -> 9.88 mm
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Other:
- board size 106.7 x 30.5 mm -> 86.4 x 27.9 mm

Commit message: update gerber && drill
Parts:
- added SW3: SW_Push, Button_Switch_THT:SW_PUSH_1P1T_6x3.5mm_H5.0_APEM_MJTP1250, F.Cu at (115.4, 121.9)
- added screw1: MountingHole_2.5mm, MountingHole:MountingHole_2.5mm, F.Cu at (108.6, 121.3)
- added screw2: MountingHole_2.5mm, MountingHole:MountingHole_2.5mm, F.Cu at (179.1, 127.0)
- BT1: footprint TestPoint:TestPoint_2Pads_Pitch5.08mm_Drill1.3mm -> Connector_PinSocket_2.54mm:PinSocket_1x02_P2.54mm_Vertical
- moved SW2 43.2 mm to (134.6, 121.9), turned to 180 degrees
- moved C2 7.50 mm to (167.7, 121.9)
- moved C1 7.07 mm to (176.5, 120.6)
- moved R1 5.08 mm to (175.3, 113.6)
- moved R2 5.08 mm to (172.7, 128.8), turned to 180 degrees
- moved J3 4.56 mm to (184.2, 121.9)
- moved J1 4.29 mm to (184.2, 128.3)
- moved BT1 3.14 mm to (160.0, 127.0), turned to 0 degrees
- moved D1 2.62 mm to (184.2, 107.3), turned to 180 degrees
- moved J2 1.39 mm to (184.2, 115.6)
- moved Q1 0.57 mm to (160.0, 115.6)
- moved SW1 0.57 mm to (162.6, 123.2)
Connections:
- U1 pad 10: unconnected-(U1-D9-Pad10) -> Net-(U1-D9)
Routing:
- net GND: track 152.0 -> 178.7 mm
- net Net-(U1-A1/D16): track 37.6 -> 18.7 mm
- net Net-(U1-A0/D15): track 32.2 -> 16.1 mm
- net Net-(U1-A2/D17): track 32.1 -> 18.7 mm
- net Net-(U1-D9): track 0.00 -> 9.03 mm
- net Net-(Q1-E): track 13.8 -> 8.43 mm
- net +9V: track 84.3 -> 89.4 mm
- net Net-(J1-PadT): track 39.8 -> 43.7 mm
- net Net-(Q1-B): track 23.9 -> 21.0 mm
- net Net-(U1-Audio_Out_1): track 45.1 -> 42.3 mm
- net Net-(D1-A): track 7.23 -> 9.55 mm
- net Net-(U1-Audio_Out_2): track 38.1 -> 37.2 mm
- added copper zone on B.Cu, net GND
- added copper zone on F.Cu, net GND
Other:
- board size 86.4 x 27.9 mm -> 86.4 x 29.2 mm
- board text added: "neum pedal v1.0 2024.01"
