File: daisy_01/daisy_01.kicad_sch (KiCad schematic)
At the start: 16 parts, among them J1 AudioInput, J2 AudioOutput1, J3 AudioOutput2, Q1 PN2222A, SW1 SW_SPST

Commit message: update
Parts:
- added SW2: RotaryEncoder_Switch, symbol Device:RotaryEncoder_Switch
- added U1: ~, symbol Electrosmith_personal:daisy_seed
- renumbered R3 to R2
Connections:
- net GND: now also SW2.C, SW2.S1; no longer A1.38 (3V3_D)
Changed lines of the file:
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@@
   (junction (at 52.07 62.23) (diameter 0) (color 0 0 0 0)
   )
+  (junction (at 175.26 138.43) (diameter 0) (color 0 0 0 0)
+  )
   (junction (at 182.88 88.9) (diameter 0) (color 0 0 0 0)
   )
@@
     (stroke (width 0) (type default))
   )
+  (wire (pts (xy 175.26 135.89) (xy 175.26 138.43))
+    (stroke (width 0) (type default))
+  )
   (wire (pts (xy 182.88 101.6) (xy 177.8 101.6))
     (stroke (width 0) (type default))
@@
     (stroke (width 0) (type default))
   )
+  (wire (pts (xy 175.26 138.43) (xy 185.42 138.43))
+    (stroke (width 0) (type default))
+  )
   (wire (pts (xy 137.16 163.83) (xy 137.16 162.56))
     (stroke (width 0) (type default))
@@
     (stroke (width 0) (type default))
   )
+  (wire (pts (xy 187.96 156.21) (xy 187.96 160.02))
+    (stroke (width 0) (type default))
+  )
   (wire (pts (xy 74.93 78.74) (xy 52.07 78.74))
     (stroke (width 0) (type default))
@@
     (stroke (width 0) (type default))
   )
+  (wire (pts (xy 175.26 138.43) (xy 175.26 160.02))
+    (stroke (width 0) (type default))
+  )
   (wire (pts (xy 187.96 104.14) (xy 215.9 104.14))
     (stroke (width 0) (type default))
@@
     (stroke (width 0) (type default))
   )
-  (wire (pts (xy 210.82 76.2) (xy 215.9 76.2))
-    (stroke (width 0) (type default))
-  )
   (wire (pts (xy 190.5 120.65) (xy 190.5 106.68))
     (stroke (width 0) (type default))
@@
     (stroke (width 0) (type default))
   )
+  (wire (pts (xy 185.42 138.43) (xy 185.42 140.97))
+    (stroke (width 0) (type default))
+  )
   (wire (pts (xy 48.26 33.02) (xy 52.07 33.02))
     (stroke (width 0) (type default))
@@
     (stroke (width 0) (type default))
   )
+  (wire (pts (xy 175.26 160.02) (xy 187.96 160.02))
+    (stroke (width 0) (type default))
+  )
   (wire (pts (xy 130.81 154.94) (xy 137.16 154.94))
     (stroke (width 0) (type default))
@@
     (effects (font (size 1.27 1.27)) (justify right))
   )
-  (hierarchical_label "GND" (shape input) (at 210.82 76.2 180) (fields_autoplaced)
-    (effects (font (size 1.27 1.27)) (justify right))
+  (hierarchical_label "GND" (shape input) (at 195.58 76.2 180) (fields_autoplaced)
+    (effects (font (size 1.27 1.27)) (justify right))
+  )
+  (hierarchical_label "GND" (shape input) (at 175.26 135.89 90) (fields_autoplaced)
+    (effects (font (size 1.27 1.27)) (justify left))
   )
   (hierarchical_label "GND" (shape input) (at 133.35 116.84 180) (fields_autoplaced)
@@
     )
   )
+  (symbol (lib_id "Device:RotaryEncoder_Switch") (at 187.96 148.59 90) (unit 1)
+    (in_bom yes) (on_board yes) (dnp no) (fields_autoplaced)
+    (property "Reference" "SW2" (at 194.31 147.32 90)
+      (effects (font (size 1.27 1.27)) (justify right))
+    )
+    (property "Value" "RotaryEncoder_Switch" (at 194.31 149.86 90)
+      (effects (font (size 1.27 1.27)) (justify right))
+    )
+    (property "Footprint" "" (at 183.896 152.4 0)
+      (effects (font (size 1.27 1.27)) hide)
+    )
+    (property "Datasheet" "~" (at 181.356 148.59 0)
+      (effects (font (size 1.27 1.27)) hide)
+    )
+    (pin "S1")
+    (pin "C")
+    (pin "B")
+    (pin "A")
+    (pin "S2")
+    (instances
+      (project "daisy_01"
+        (path "/e8113027-a6e3-419d-b0ee-bd8e9fb4b03a"
+          (reference "SW2") (unit 1)
+        )
+      )
+    )
+  )
+  (symbol (lib_id "Electrosmith_personal:daisy_seed") (at 71.12 110.49 0) (unit 1)
+    (in_bom yes) (on_board yes) (dnp no) (fields_autoplaced)
+    (property "Reference" "U1" (at 71.12 102.87 0)
+      (effects (font (size 1.27 1.27)))
+    )
+    (property "Value" "~" (at 59.69 110.49 0)
+      (effects (font (size 1.27 1.27)))
+    )
+    (property "Footprint" "" (at 59.69 110.49 0)
+      (effects (font (size 1.27 1.27)) hide)
+    )
+    (property "Datasheet" "" (at 59.69 110.49 0)
+      (effects (font (size 1.27 1.27)) hide)
+    )
+    (pin "24")
+    (pin "11")
+    (pin "28")
+    (pin "20")
+    (pin "30")
+    (pin "40")
+    (pin "31")
+    (pin "6")
+    (pin "9")
+    (pin "35")
+    (pin "32")
+    (pin "29")
+    (pin "3")
+    (pin "21")
+    (pin "8")
+    (pin "14")
+    (pin "15")
+    (pin "33")
+    (pin "16")
+    (pin "37")
+    (pin "1")
+    (pin "39")
+    (pin "13")
+    (pin "12")
+    (pin "10")
+    (pin "26")
+    (pin "38")
+    (pin "27")
+    (pin "4")
+    (pin "34")
+    (pin "5")
+    (pin "25")
+    (pin "7")
+    (pin "22")
+    (pin "2")
+    (pin "19")
+    (pin "17")
+    (pin "23")
+    (pin "36")
+    (pin "18")
+    (instances
+      (project "daisy_01"
+        (path "/e8113027-a6e3-419d-b0ee-bd8e9fb4b03a"
+          (reference "U1") (unit 1)
+        )
+      )
+    )
+  )
   (symbol (lib_id "Connector_Audio:AudioJack2") (at 172.72 91.44 0) (unit 1)
     (in_bom yes) (on_board yes) (dnp no) (fields_autoplaced)
@@
   (symbol (lib_id "Device:R") (at 74.93 41.91 180) (unit 1)
     (in_bom yes) (on_board yes) (dnp no) (fields_autoplaced)
-    (property "Reference" "R3" (at 77.47 40.64 0)
+    (property "Reference" "R2" (at 77.47 40.64 0)
       (effects (font (size 1.27 1.27)) (justify right))
     )
@@
       (project "daisy_01"
         (path "/e8113027-a6e3-419d-b0ee-bd8e9fb4b03a"
-          (reference "R3") (unit 1)
-        )
-      )
+          (reference "R2") (unit 1)
+        )
+      )

Commit message: update
Parts:
- removed A1: Device_Audio_Electrosmith_Daisy_Seed_Rev4, Daisy_Electrosmith:Device_Audio_Electrosmith_Daisy_Seed, symbol test_daisy:Device_Audio_Electrosmith_Daisy_Seed_Rev4
- SW2: footprint (none) -> Rotary_Encoder:RotaryEncoder_Alps_EC11E-Switch_Vertical_H20mm
- U1: footprint (none) -> Library_electrosmith:Device_Audio_Electrosmith_Daisy_Seed
Connections:
- net +9V: now also U1.39 (VIN)
- net A_PWR3.3: now also U1.21 (3V3_ANALOG)
- net GND: now also U1.20 (AGND), U1.40 (DGND)
- net at J1.T: now also U1.16 (Audio_In_1)
- net at J2.T: now also U1.18 (Audio_Out_1)
- net at J3.T: now also U1.19 (Audio_Out_2)
- net at RV1.2: now also U1.25 (A3/D18)
- net at RV2.2: now also U1.26 (A4/D19)
- net at RV3.2: now also U1.27 (A5/D20)
- net at RV4.2: now also U1.28 (A5/D21)
- net at SW2.A: now also U1.22 (A0/D15)
- net at SW2.B: now also U1.23 (A1/D16)
- net at SW2.S2: now also U1.24 (A2/D17)
Other:
- moved on the sheet: J1, J2, J3, RV1, RV2, RV3, RV4, SW2, U1

Commit message: update
Connections:
- net A_PWR3.3: now also RV1.3, RV2.3, RV3.3, RV4.3; no longer RV1.1, RV2.1, RV3.1, RV4.1
- net GND: now also RV1.1, RV2.1, RV3.1, RV4.1; no longer RV1.3, RV2.3, RV3.3, RV4.3
Changed lines of the file:
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@@
     (effects (font (size 1.27 1.27)) (justify right))
   )
-  (hierarchical_label "A_PWR3.3" (shape input) (at 228.6 128.27 0) (fields_autoplaced)
+  (hierarchical_label "A_PWR3.3" (shape input) (at 228.6 119.38 0) (fields_autoplaced)
     (effects (font (size 1.27 1.27)) (justify left))
   )
-  (hierarchical_label "A_PWR3.3" (shape input) (at 226.06 83.82 0) (fields_autoplaced)
+  (hierarchical_label "A_PWR3.3" (shape input) (at 226.06 71.12 0) (fields_autoplaced)
     (effects (font (size 1.27 1.27)) (justify left))
   )
@@
     (effects (font (size 1.27 1.27)) (justify right))
   )
-  (hierarchical_label "GND" (shape input) (at 226.06 71.12 0) (fields_autoplaced)
+  (hierarchical_label "GND" (shape input) (at 226.06 83.82 0) (fields_autoplaced)
     (effects (font (size 1.27 1.27)) (justify left))
   )
-  (hierarchical_label "GND" (shape input) (at 228.6 119.38 0) (fields_autoplaced)
+  (hierarchical_label "GND" (shape input) (at 228.6 128.27 0) (fields_autoplaced)
     (effects (font (size 1.27 1.27)) (justify left))
   )
@@
     (effects (font (size 1.27 1.27)) (justify left))
   )
-  (hierarchical_label "GND" (shape input) (at 228.6 104.14 0) (fields_autoplaced)
+  (hierarchical_label "GND" (shape input) (at 228.6 113.03 0) (fields_autoplaced)
     (effects (font (size 1.27 1.27)) (justify left))
   )
@@
     (effects (font (size 1.27 1.27)) (justify right))
   )
-  (hierarchical_label "A_PWR3.3" (shape input) (at 227.33 99.06 0) (fields_autoplaced)
+  (hierarchical_label "A_PWR3.3" (shape input) (at 226.06 88.9 0) (fields_autoplaced)
     (effects (font (size 1.27 1.27)) (justify left))
   )
-  (hierarchical_label "A_PWR3.3" (shape input) (at 228.6 113.03 0) (fields_autoplaced)
+  (hierarchical_label "A_PWR3.3" (shape input) (at 228.6 104.14 0) (fields_autoplaced)
     (effects (font (size 1.27 1.27)) (justify left))
   )
@@
     (effects (font (size 1.27 1.27)) (justify left))
   )
-  (hierarchical_label "GND" (shape input) (at 226.06 88.9 0) (fields_autoplaced)
+  (hierarchical_label "GND" (shape input) (at 227.33 99.06 0) (fields_autoplaced)
     (effects (font (size 1.27 1.27)) (justify left))
   )

Commit message: update
Parts:
- SW2: footprint Rotary_Encoder:RotaryEncoder_Alps_EC11E-Switch_Vertical_H20mm -> personal_footprints:ec11_encoder_mio
Changed lines of the file:
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@@
       (effects (font (size 1.27 1.27)))
     )
-    (property "Footprint" "Rotary_Encoder:RotaryEncoder_Alps_EC11E-Switch_Vertical_H20mm" (at 223.52 51.816 0)
+    (property "Footprint" "personal_footprints:ec11_encoder_mio" (at 223.52 51.816 0)
       (effects (font (size 1.27 1.27)) hide)
     )

Commit message: update gerber && drill
Parts:
- added SW3: SW_Push, Button_Switch_THT:SW_PUSH_1P1T_6x3.5mm_H5.0_APEM_MJTP1250, symbol Switch:SW_Push
- BT1: footprint TestPoint:TestPoint_2Pads_Pitch5.08mm_Drill1.3mm -> Connector_PinSocket_2.54mm:PinSocket_1x02_P2.54mm_Vertical
Connections:
- net GND: now also SW3.1
- net at U1.10 (D9): now also SW3.2
